File: BE6502 Mega Adapter/BE6502 Mega Adapter.kicad_pcb (KiCad board)
At the start: 2 copper layers, 99.1 x 99.1 mm, 12 parts, among them J1 Expansion, J2 Slot #1, J3 Slot #2, M1 Mounting, M2 Mounting, M3 Mounting, M4 Mounting

Commit message: Added some switches and an LED to unused pins
Parts:
- added D1: USER, LEDs:LED_D5.0mm, F.Cu at (114.3, 123.4)
- added R1: 10k, Resistors_THT:R_Axial_DIN0207_L6.3mm_D2.5mm_P10.16mm_Horizontal, F.Cu at (158.1, 118.7)
- added R2: 10k, Resistors_THT:R_Axial_DIN0207_L6.3mm_D2.5mm_P10.16mm_Horizontal, F.Cu at (158.1, 121.9)
- added R3: 10k, Resistors_THT:R_Axial_DIN0207_L6.3mm_D2.5mm_P10.16mm_Horizontal, F.Cu at (158.1, 125.1)
- added R4: 220, Resistors_THT:R_Axial_DIN0207_L6.3mm_D2.5mm_P10.16mm_Horizontal, F.Cu at (119.4, 129.5)
- added SW1: SW_Push, Buttons_Switches_THT:SW_PUSH_6mm, F.Cu at (120.7, 120.0)
- added SW2: SW_Push, Buttons_Switches_THT:SW_PUSH_6mm, F.Cu at (131.4, 120.0)
- added SW3: SW_Push, Buttons_Switches_THT:SW_PUSH_6mm, F.Cu at (142.2, 120.0)
Connections:
- XA1 pad A10: (no net) -> Net-(R3-Pad1)
- XA1 pad A11: (no net) -> Net-(D1-Pad2)
- XA1 pad A8: (no net) -> Net-(R1-Pad1)
- XA1 pad A9: (no net) -> Net-(R2-Pad1)
Routing:
- net Net-(D1-Pad2): track 0.00 -> 80.9 mm, vias 0 -> 4
- net Net-(R1-Pad1): track 0.00 -> 66.5 mm, vias 0 -> 1
- net Net-(R2-Pad1): track 0.00 -> 52.4 mm, vias 0 -> 1
- net Net-(R3-Pad1): track 0.00 -> 39.1 mm, vias 0 -> 1
- net VCC: track 153.1 -> 186.5 mm, vias 2 -> 3
- net Net-(D1-Pad1): track 0.00 -> 10.1 mm, vias 0 -> 1
- net /CLOCK: track 106.1 -> 109.4 mm
- net /D2: track 165.3 -> 167.1 mm
- net /D1: track 164.7 -> 166.3 mm
- net /D7: track 174.0 -> 175.5 mm
- net /D5: track 167.1 -> 168.7 mm
- net /D0: track 164.1 -> 165.3 mm
- net /~RDY: track 97.8 -> 99.0 mm
- net /A0: track 155.6 -> 156.6 mm
- net /~NMI: track 95.7 -> 96.7 mm
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Other:
- board text added: "Revision B"
- board text added: "User-definable functions"
- board text removed: "Revision A"
