File: BE6502 Clock/BE6502 Clock.sch (KiCad schematic (older format))
At the start: 28 parts, among them J1 CLOCK_SEL, M1 Mounting, M2 Mounting, M3 Mounting, M4 Mounting, SW1 MANUAL, SW2 CLK_SEL, U1 LM555, U2 LM555, U3 LM555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

Commit message: Updated clock with capacitor from video 3
Parts:
- added C8: 100nF, Capacitors_THT:C_Disc_D4.7mm_W2.5mm_P5.00mm, symbol C
Connections:
- net GND: now also C8.2
- net at R3.2, SW1.2, U2.2 (TR): now also C8.1
Other:
- note added: "B"
- note removed: "A"
- moved on the sheet: SW1
